File: rear-projection-display/rear-projection-display.kicad_pcb (KiCad board)
At the start: 2 copper layers, 49.9 x 35.7 mm, 21 parts, among them J1 QWIIC, J2 +5V Power, U1 IS31FL3236A-QFLS2-TR

Commit message: Add interior housing hole cutout to board outline
Adds a 2.25mm-radius circular cutout on Edge.Cuts at (166.09, 95.36)
per the updated board outline DXF. Corresponds to DXF position
(12.64, 6.005) relative to board center.

Co-Authored-By: Claude Sonnet 4.6 <noreply@anthropic.com>
Parts:
- moved R1 17.6 mm to (153.4, 91.0)
- moved C1 13.5 mm to (150.9, 108.5), turned to 90 degrees
- moved C2 13.1 mm to (157.6, 108.6), turned to 90 degrees
- moved R2 0.08 mm to (141.6, 106.5)
Routing:
- net GND: track 0.00 -> 148.7 mm
Other:
- outline, holes or cut-outs redrawn
Changed lines of the file:
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@@
 		(tags "LED RGB 10mm through-hole")
 		(property "Reference" "D6"
-			(at 0 -7 0)
+			(at -0.075 -2.525 0)
 			(layer "F.SilkS")
 			(effects
@@
 			(at 8.2 -10.795 0)
 			(layer "B.Cu")
+			(hide yes)
 			(effects
 				(font
@@
 		(tags "LED RGB 10mm through-hole")
 		(property "Reference" "D7"
-			(at 0 -7 0)
+			(at 0.075 -2.325 0)
 			(layer "F.SilkS")
 			(effects
@@
 		(tags "LED RGB 10mm through-hole")
 		(property "Reference" "D12"
-			(at 0 -7 0)
+			(at -0.075 -2.525 0)
 			(layer "F.SilkS")
 			(effects
@@
 		(tags "LED RGB 10mm through-hole")
 		(property "Reference" "D9"
-			(at 0 -7 0)
+			(at -0.225 -2.525 0)
 			(layer "F.SilkS")
 			(effects
@@
 			(at 8.2 -10.795 0)
 			(layer "B.Cu")
+			(hide yes)
 			(effects
 				(font
@@
 		(tags "LED RGB 10mm through-hole")
 		(property "Reference" "D5"
-			(at 0 -7 0)
+			(at 0.025 -2.475 0)
 			(layer "F.SilkS")
 			(effects
@@
 		(tags "LED RGB 10mm through-hole")
 		(property "Reference" "D10"
-			(at 0 -7 0)
+			(at -0.175 -2.425 0)
 			(layer "F.SilkS")
 			(effects
@@
 		(tags "LED RGB 10mm through-hole")
 		(property "Reference" "D2"
-			(at 0 -7 0)
+			(at -0.025 -2.475 0)
 			(layer "F.SilkS")
 			(effects
@@
 		(tags "LED RGB 10mm through-hole")
 		(property "Reference" "D3"
-			(at 0 -7 0)
+			(at 0.075 -2.425 0)
 			(layer "F.SilkS")
 			(effects
@@
 			(at 8.2 -10.795 0)
 			(layer "B.Cu")
+			(hide yes)
 			(effects
 				(font
@@
 		(tags "LED RGB 10mm through-hole")
 		(property "Reference" "D4"
-			(at 0 -7 0)
+			(at 0.025 -2.625 0)
 			(layer "F.SilkS")
 			(effects
@@
 		(tags "LED RGB 10mm through-hole")
 		(property "Reference" "D1"
-			(at 0 -7 0)
+			(at 0 -2.525 0)
 			(layer "F.SilkS")
 			(effects
@@
 		(tags "LED RGB 10mm through-hole")
 		(property "Reference" "D11"
-			(at 0 -7 0)
+			(at -0.075 -2.675 0)
 			(layer "F.SilkS")
 			(effects
@@
 		(tags "LED RGB 10mm through-hole")
 		(property "Reference" "D8"
-			(at 0 -7 0)
+			(at 0.075 -2.375 0)
 			(layer "F.SilkS")
 			(effects
@@
 	(footprint "Resistor_SMD:R_0603_1608Metric"
 		(layer "B.Cu")
-		(at 141.5 106.49 180)
+		(at 141.575 106.5 180)
 		(descr "Resistor SMD 0603 (1608 Metric), square (rectangular) end terminal, IPC-7351 nominal, (Body size source: IPC-SM-782 page 72, https://www.pcb-3d.com/wordpress/wp-content/uploads/ipc-sm-782a_amendment_1_and_2.pdf)")
 		(tags "resistor")
@@
 	(footprint "Capacitor_SMD:C_0805_2012Metric"
 		(layer "B.Cu")
-		(at 160.95 96 180)
+		(at 157.6 108.625 90)
 		(descr "Capacitor SMD 0805 (2012 Metric), square (rectangular) end terminal, IPC-7351 nominal, (Body size source: IPC-SM-782 page 76, https://www.pcb-3d.com/wordpress/wp-content/uploads/ipc-sm-782a_amendment_1_and_2.pdf, https://docs.google.com/spreadsheets/d/1BsfQQcO9C6DZCsRaXUlFlo91Tg2WpOkGARC1WS5S8t0/edit?usp=sharing)")
 		(tags "capacitor")
 		(property "Reference" "C2"
-			(at 0 1.68 0)
+			(at 0.025 2.375 90)
 			(layer "B.SilkS")
 			(effects
@@
 		)
 		(property "Value" "10uF"
-			(at 0 -1.68 0)
+			(at 0 -1.68 90)
 			(layer "B.Fab")
 			(effects
@@
 		)
 		(property "Datasheet" ""
-			(at 0 0 0)
+			(at 0 0 90)
 			(layer "B.Fab")
 			(hide yes)
@@
 		)
 		(property "Description" ""
-			(at 0 0 0)
+			(at 0 0 90)
 			(layer "B.Fab")
 			(hide yes)
@@
 		)
 		(property "KiLib_Generator" "SMD_2terminal_chip_molded"
-			(at 0 0 0)
+			(at 0 0 90)
 			(layer "B.SilkS")
 			(hide yes)
@@
 		(duplicate_pad_numbers_are_jumpers no)
 		(fp_line
-			(start -0.261252 0.735)
-			(end 0.261252 0.735)
+			(start -0.261252 -0.735)
+			(end 0.261252 -0.735)
 			(stroke
 				(width 0.12)
@@
 		)
 		(fp_line
-			(start -0.261252 -0.735)
-			(end 0.261252 -0.735)
+			(start -0.261252 0.735)
+			(end 0.261252 0.735)
 			(stroke
 				(width 0.12)
@@
 		)
 		(fp_text user "${REFERENCE}"
-			(at 0 0 0)
+			(at -2.85 0.2 90)
 			(layer "B.Fab")
 			(effects
@@
 		)
 		(pad "1" smd roundrect
-			(at -0.95 0 180)
+			(at -0.95 0 90)
 			(size 1 1.45)
 			(layers "B.Cu" "B.Mask" "B.Paste")
@@
 		)
 		(pad "2" smd roundrect
-			(at 0.95 0 180)
+			(at 0.95 0 90)
 			(size 1 1.45)
 			(layers "B.Cu" "B.Mask" "B.Paste")
@@
 	(footprint "Resistor_SMD:R_0603_1608Metric"
 		(layer "B.Cu")
-		(at 141.5 103.98 180)
+		(at 153.375 91 180)
 		(descr "Resistor SMD 0603 (1608 Metric), square (rectangular) end terminal, IPC-7351 nominal, (Body size source: IPC-SM-782 page 72, https://www.pcb-3d.com/wordpress/wp-content/uploads/ipc-sm-782a_amendment_1_and_2.pdf)")
 		(tags "resistor")
@@
 	(footprint "Capacitor_SMD:C_0402_1005Metric"
 		(layer "B.Cu")
-		(at 164.165 105.85 180)
+		(at 150.9 108.5 90)
 		(descr "Capacitor SMD 0402 (1005 Metric), square (rectangular) end terminal, IPC-7351 nominal, (Body size source: IPC-SM-782 page 76, https://www.pcb-3d.com/wordpress/wp-content/uploads/ipc-sm-782a_amendment_1_and_2.pdf)")
 		(tags "capacitor")
 		(property "Reference" "C1"
-			(at 10.665 4.85 0)
+			(at -0.295 -1.925 90)
 			(layer "B.SilkS")
 			(effects
@@
 		)
 		(property "Value" "100nF"
-			(at 0 -1.16 0)
+			(at 0 -1.16 90)
 			(layer "B.Fab")
+			(hide yes)
 			(effects
 				(font
@@
 		)
 		(property "Datasheet" ""
-			(at 0 0 0)
+			(at 0 0 90)
 			(layer "B.Fab")
 			(hide yes)
@@
 		)
 		(property "Description" ""
-			(at 0 0 0)
+			(at 0 0 90)
 			(layer "B.Fab")
 			(hide yes)
@@
 		)
 		(property "KiLib_Generator" "SMD_2terminal_chip_molded"
-			(at 0 0 0)
+			(at 0 0 90)
 			(layer "B.SilkS")
 			(hide yes)
@@
 		(duplicate_pad_numbers_are_jumpers no)
 		(fp_line
-			(start -0.107836 0.36)
-			(end 0.107836 0.36)
+			(start -0.107836 -0.36)
+			(end 0.107836 -0.36)
 			(stroke
 				(width 0.12)
@@
 		)
 		(fp_line
-			(start -0.107836 -0.36)
-			(end 0.107836 -0.36)
+			(start -0.107836 0.36)
+			(end 0.107836 0.36)
 			(stroke
 				(width 0.12)
@@
 		)
 		(fp_text user "${REFERENCE}"
-			(at 0 0 0)
+			(at 0 0 90)
 			(layer "B.Fab")
 			(effects
@@
 		)
 		(pad "1" smd roundrect
-			(at -0.48 0 180)
+			(at -0.48 0 90)
 			(size 0.56 0.62)
 			(layers "B.Cu" "B.Mask" "B.Paste")
@@
 		)
 		(pad "2" smd roundrect
-			(at 0.48 0 180)
+			(at 0.48 0 90)
 			(size 0.56 0.62)
 			(layers "B.Cu" "B.Mask" "B.Paste")
@@
 		(layer "Edge.Cuts")
 	)
+	(gr_circle
+		(center 166.09 95.36)
+		(end 168.34 95.36)
+		(stroke
+			(width 0.1)
+			(type default)
+		)
+		(fill none)
+		(layer "Edge.Cuts")
+	)
+	(segment
+		(start 154 106.095)
+		(end 137.43 89.525)
+		(width 0.2)
+		(layer "F.Cu")
+		(net "GND")
+	)
+	(segment
+		(start 162.33 90.325)
+		(end 161.53 89.525)
+		(width 0.2)
+		(layer "F.Cu")
+		(net "GND")
+	)
+	(segment
+		(start 173.58 113.625)
+		(end 173.58 101.575)
+		(width 0.2)
+		(layer "F.Cu")
+		(net "GND")
+	)
+	(segment
+		(start 162.33 114.425)
+		(end 172.78 114.425)
+		(width 0.2)
+		(layer "F.Cu")
+		(net "GND")
+	)
+	(segment
+		(start 137.43 89.525)
+		(end 138.23 90.325)
+		(width 0.2)
+		(layer "F.Cu")
+		(net "GND")
+	)
+	(segment
+		(start 173.58 89.525)
+		(end 172.78 90.325)
+		(width 0.2)
+		(layer "F.Cu")
+		(net "GND")
+	)
+	(segment
+		(start 160.73 114.425)
+		(end 161.53 113.625)
+		(width 0.2)
+		(layer "F.Cu")
+		(net "GND")
+	)
+	(segment
+		(start 148.68 90.325)
+		(end 149.48 89.525)
+		(width 0.2)
+		(layer "F.Cu")
+		(net "GND")
+	)
+	(segment
+		(start 149.48 113.625)
+		(end 150.28 114.425)
+		(width 0.2)
+		(layer "F.Cu")
+		(net "GND")
+	)
+	(segment
+		(start 161.53 101.575)
+		(end 161.53 89.525)
+		(width 0.2)
+		(layer "F.Cu")
+		(net "GND")
+	)
+	(segment
+		(start 137.43 101.575)
+		(end 137.43 89.525)
+		(width 0.2)
+		(layer "F.Cu")
+		(net "GND")
+	)
+	(segment
+		(start 161.53 113.625)
+		(end 162.33 114.425)
+		(width 0.2)
+		(layer "F.Cu")
+		(net "GND")
+	)
+	(segment
+		(start 150.28 114.425)
+		(end 160.73 114.425)
+		(width 0.2)
+		(layer "F.Cu")
+		(net "GND")
+	)
+	(segment
+		(start 137.43 101.575)
+		(end 137.43 113.625)
+		(width 0.2)
+		(layer "F.Cu")
+		(net "GND")
+	)
+	(segment
+		(start 137.43 113.625)
+		(end 138.23 114.425)
+		(width 0.2)
+		(layer "F.Cu")
+		(net "GND")
+	)
+	(segment
+		(start 154 107.5)
+		(end 154 106.095)
+		(width 0.2)
+		(layer "F.Cu")
+		(net "GND")
+	)
+	(segment
+		(start 138.23 114.425)
+		(end 148.68 114.425)
+		(width 0.2)
+		(layer "F.Cu")
+		(net "GND")
+	)
+	(segment
+		(start 173.58 101.575)
+		(end 173.58 89.525)
+		(width 0.2)
+		(layer "F.Cu")
+		(net "GND")
+	)
+	(segment
+		(start 172.78 90.325)
+		(end 162.33 90.325)
+		(width 0.2)
+		(layer "F.Cu")
+		(net "GND")
+	)
+	(segment
+		(start 148.68 114.425)
+		(end 149.48 113.625)
+		(width 0.2)
+		(layer "F.Cu")
+		(net "GND")
+	)
+	(segment
+		(start 172.78 114.425)
+		(end 173.58 113.625)
+		(width 0.2)
+		(layer "F.Cu")
+		(net "GND")
+	)
+	(segment
+		(start 138.23 90.325)
+		(end 148.68 90.325)
+		(width 0.2)
+		(layer "F.Cu")
+		(net "GND")
+	)
 	(group ""
