File: led-indicator/led-indicator/led-indicator.kicad_pcb (KiCad board)
At the start: 2 copper layers, 49.9 x 35.7 mm, 33 parts, among them CN1 XT30UPB-F, J2 JST_XH_3pin, U1 74AHCT125

Commit message: led-indicator: PCB fixes, +5V trace widening, datasheet and CN1 reconciliation
PCB fixes:
- PM-001: Move C8 to (161.7, 102.8) and C12 to (161.7, 114.8) — aligned
  with C4 pattern, to the left of D8/D12 instead of to the right where the
  LED courtyard and board edge left no valid placement zone
- PM-002: Move FID2 to (169.35, 87.85) — 3mm inset from corner clears the
  Fiducial_1mm_Mask2mm courtyard from the board edge
- FD-001: Add FID4/FID5/FID6 on B.Cu at 3mm inset from corners to support
  back-side SMD assembly pass (U1 SOIC-14, R1 0603, SJ1 solder jumper)
- XV-002: Update PCB D1 value to "SK6812RGBW" to match schematic

+5V trace widening:
- All 96 +5V segments (F.Cu and B.Cu) widened from 0.2mm to 0.8mm
- 0.8mm supports ~1.5A on outer layer (10°C rise, 1oz Cu), sufficient
  margin for 720mA peak load at full-white across 12 SK6812 LEDs
- "Power" net class created (0.8mm trace, 0.3mm clearance) to enforce
  width on future edits
- GND return path handled by the full-board copper pours added previously

CN1 reconciliation:
- Confirmed CN1 (XT30UPB-F power connector) is correctly present in both
  schematic (UUID 7c51e3ce, output pins on +5V and GND) and PCB
  (pad1=+5V, pad2=GND, B.Cu); the XV-001 "extra in PCB" finding was a
  false positive caused by the JLC symbol using (power local) flag which
  the cross-analyzer excludes from component matching

Datasheet:
- D1–D12 Datasheet property set to SK6812RGBW Rev.01 datasheet
  (via Adafruit CDN, the canonical distribution source for this part)

Co-Authored-By: Claude Sonnet 4.6 <noreply@anthropic.com>
Parts:
- added FID4: Fiducial_1mm_Mask2mm, Fiducial:Fiducial_1mm_Mask2mm, B.Cu at (125.3, 87.8)
- added FID5: Fiducial_1mm_Mask2mm, Fiducial:Fiducial_1mm_Mask2mm, B.Cu at (169.3, 87.8)
- added FID6: Fiducial_1mm_Mask2mm, Fiducial:Fiducial_1mm_Mask2mm, B.Cu at (125.3, 117.7)
- D1: value 12x SK6812RGBW -> SK6812RGBW
- moved C12 7.70 mm to (161.7, 114.8)
- moved C8 7.60 mm to (161.7, 102.8)
- moved FID2 1.41 mm to (169.3, 87.8)

Commit message: led-indicator: manual rerouting and schematic edits
Manual PCB re-routing after previous trace-width widening caused
clearance violations. Includes schematic updates made during the same
editing session. Also removes stale LED board layout DXF and updates
the board outline DXF.

Co-Authored-By: Claude Sonnet 4.6 <noreply@anthropic.com>
Parts:
- removed FID1, FID2, FID3, FID4, FID5, FID6: Fiducial_1mm_Mask2mm, Fiducial:Fiducial_1mm_Mask2mm
- moved R1 1.61 mm to (128.8, 89.3)
Connections:
- net Net-(D10-DIN) renamed /D_9_10
- net Net-(D10-DOUT) renamed /D_10_11
- net Net-(D11-DOUT) renamed /D_11_12
- net Net-(D3-DOUT) renamed /D_3_4
- net Net-(D4-DOUT) renamed /D_4_5
- net Net-(D5-DOUT) renamed /D_5_6
- net Net-(D6-DOUT) renamed /D_6_7
- net Net-(D7-DOUT) renamed /D_7_8
- net Net-(D8-DOUT) renamed /D_8_9
- D1 pad 4: Net-(D1-DOUT) -> /D_1_2
- D2 pad 2: Net-(D1-DOUT) -> /D_1_2
- D2 pad 4: Net-(D1-DOUT) -> /D_2_3
- D3 pad 2: Net-(D1-DOUT) -> /D_2_3
- R1 pad 1: Net-(R1-Pad1) -> /DIN_5V
- R1 pad 2: /DIN -> Net-(R1-Pad2)
- U1 pad 2: Net-(R1-Pad1) -> /DIN
- U1 pad 3: /DIN_5V -> Net-(R1-Pad2)
Routing:
- net GND: track 244.9 -> 21.5 mm, vias 3 -> 10
- net /DIN: track 20.6 -> 47.9 mm
- net +5V: track 218.8 -> 243.9 mm, vias 1 -> 0
- net /DIN_5V: track 29.3 -> 4.82 mm
- net Net-(R1-Pad2): track 0.00 -> 24.1 mm
- net Net-(R1-Pad1): track 20.6 -> 0.00 mm
- net Net-(D1-DOUT): track 18.6 -> 0.00 mm
- net /D_1_2: track 0.00 -> 9.08 mm
- net /D_2_3: track 0.00 -> 9.03 mm
- net /D_4_5: track 54.5 -> 60.0 mm

Commit message: led-indicator: add fiducials for double-sided SMD assembly
Place 6 Fiducial_0.5mm_Mask1mm footprints for JLCPCB pick-and-place
alignment — 3 on F.Cu (REF01/02/03) and 3 on B.Cu (REF04/05/06) near
board corners. DRC clean: 0 violations, 0 unconnected.

Co-Authored-By: Claude Sonnet 4.6 <noreply@anthropic.com>
Parts:
- added REF01: Fiducial_0.5mm_Mask1mm, Fiducial:Fiducial_0.5mm_Mask1mm, F.Cu at (126.0, 86.7)
- added REF02: Fiducial_0.5mm_Mask1mm, Fiducial:Fiducial_0.5mm_Mask1mm, F.Cu at (169.2, 86.6)
- added REF03: Fiducial_0.5mm_Mask1mm, Fiducial:Fiducial_0.5mm_Mask1mm, F.Cu at (127.4, 118.5)
- added REF04: Fiducial_0.5mm_Mask1mm, Fiducial:Fiducial_0.5mm_Mask1mm, B.Cu at (170.1, 87.2)
- added REF05: Fiducial_0.5mm_Mask1mm, Fiducial:Fiducial_0.5mm_Mask1mm, B.Cu at (170.1, 118.4)
- added REF06: Fiducial_0.5mm_Mask1mm, Fiducial:Fiducial_0.5mm_Mask1mm, B.Cu at (124.8, 118.6)

Commit message: led-indicator: replace CN1 with XT30U-M (male) connector
Switch CN1 from XT30UPB-F (female, C108769) to XT30U-M (male, C99101).
The male connector mates with the battery's female harness plug.

Updated both schematic and PCB:
- Footprint: AMASS_XT30UPB-F → AMASS_XT30U-M (drill 1.8mm → 2.7mm,
  pad size 3×3mm → 3.8×3.8mm, roundrect ratio 0.25 → 0.2)
- LCSC Part: C108769 → C99101
- MPN: XT30UPB-F30.G.Y → XT30U-M
- Refilled copper zones after pad size change; DRC clean (0 errors,
  0 unconnected — only pre-existing C7 library mismatch warning remains)

Co-Authored-By: Claude Sonnet 4.6 <noreply@anthropic.com>
Parts:
- CN1: value XT30UPB-F -> XT30U-M; footprint Connector_AMASS:AMASS_XT30UPB-F_1x02_P5.0mm_Vertical -> Connector_AMASS:AMASS_XT30U-M_1x02_P5.0mm_Vertical
Changed lines of the file:
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@@
 			(size 0.9 0.95)
 			(layers "F.Cu" "F.Mask" "F.Paste")
-			(roundrect_rratio 0.25)
+			(roundrect_rratio 0.2)
 			(net "+5V")
 			(pintype "passive")
@@
 		)
 	)
-	(footprint "Connector_AMASS:AMASS_XT30UPB-F_1x02_P5.0mm_Vertical"
+	(footprint "Connector_AMASS:AMASS_XT30U-M_1x02_P5.0mm_Vertical"
 		(layer "B.Cu")
 		(at 162.3 108.625 180)
-		(descr "Connector XT30 Vertical PCB Female, https://www.tme.eu/Document/81f11ca924696756331f21b972812074/XT30PB-F.pdf")
+		(descr "Connector XT30 Vertical Cable Male, https://www.tme.eu/Document/7d9d972ae3468777f69ec2ee99897652/XT30U-M.pdf")
 		(tags "RC Connector XT30")
 		(property "Reference" "CN1"
@@
 			)
 		)
-		(property "Value" "XT30UPB-F"
+		(property "Value" "XT30U-M"
 			(at 2.5 -4 0)
 			(layer "B.Fab")
@@
 			)
 		)
-		(property "Datasheet" "https://lcsc.com/product-detail/Banana-and-Tip-Connectors_Changzhou-Amass-Elec-XT30UPB-F_C108769.html"
+		(property "Datasheet" "https://www.lcsc.com/product-detail/C99101.html"
 			(at 0 0 0)
 			(unlocked yes)
@@
 			)
 		)
-		(property "MPN" "XT30UPB-F30.G.Y"
+		(property "MPN" "XT30U-M"
 			(at 0 0 0)
 			(unlocked yes)
@@
 			)
 		)
-		(property "LCSC Part" "C108769"
+		(property "LCSC Part" "C99101"
 			(at 0 0 0)
 			(unlocked yes)
@@
 		(pad "1" thru_hole roundrect
 			(at 0 0 180)
-			(size 3 3)
-			(drill 1.8)
+			(size 3.8 3.8)
+			(drill 2.7)
 			(layers "*.Cu" "*.Mask")
 			(remove_unused_layers no)
-			(roundrect_rratio 0.25)
+			(roundrect_rratio 0.2)
 			(net "+5V")
 			(pinfunction "+_1")
@@
 		(pad "2" thru_hole circle
 			(at 5 0 180)
-			(size 3 3)
-			(drill 1.8)
+			(size 3.8 3.8)
+			(drill 2.7)
 			(layers "*.Cu" "*.Mask")
 			(remove_unused_layers no)
@@
 		)
 		(embedded_fonts no)
-		(model "${KICAD10_3DMODEL_DIR}/Connector_AMASS.3dshapes/AMASS_XT30UPB-F_1x02_P5.0mm_Vertical.step"
+		(model "${KICAD10_3DMODEL_DIR}/Connector_AMASS.3dshapes/AMASS_XT30U-M_1x02_P5.0mm_Vertical.step"
 			(offset
 				(xyz 0 0 0)
