File: led-indicator/led-indicator/led-indicator.kicad_sch (KiCad schematic)
At the start: 29 parts, among them J2 JST_XH_3pin, U1 74AHCT125

Commit message: led-indicator: manual rerouting and schematic edits
Manual PCB re-routing after previous trace-width widening caused
clearance violations. Includes schematic updates made during the same
editing session. Also removes stale LED board layout DXF and updates
the board outline DXF.

Co-Authored-By: Claude Sonnet 4.6 <noreply@anthropic.com>
Connections:
- net D_3_4: now reaches D3.4 (DOUT), D4.2 (DIN)
- net D_4_5: now reaches D4.4 (DOUT), D5.2 (DIN)
- net D_8_9: now reaches D8.4 (DOUT), D9.2 (DIN)
- net D_9_10: now reaches D10.2 (DIN), D9.4 (DOUT)
- net D_1_2: now reaches D1.4 (DOUT), D2.2 (DIN)
- net D_2_3: now reaches D2.4 (DOUT), D3.2 (DIN)
- net D_10_11: now reaches D10.4 (DOUT), D11.2 (DIN)
- net D_11_12: now reaches D11.4 (DOUT), D12.2 (DIN)
- net D_6_7: now reaches D6.4 (DOUT), D7.2 (DIN)
- net D_7_8: now reaches D7.4 (DOUT), D8.2 (DIN)
- net D_5_6: now reaches D5.4 (DOUT), D6.2 (DIN)

Commit message: led-indicator: add LCSC/MPN part numbers to all BOM components
Sets LCSC and MPN hidden properties on all 29 purchasable components
for JLCPCB assembly ordering:

  C1-C12   C14663     CC0603KRX7R9BB104     100nF 0603 (Basic)
  C13      C3299      GR108M010F12RR0VL4FP0 1000uF 10V radial THT
  D1-D12   C22464516  XL-5050RGBWC-WS2812B  SK6812-compat 5050 RGBW
  J2       C144394    B3B-XH-A(LF)(SN)      JST XH 3-pin
  R1       C23138     0603WAF3300T5E         330R 0603 (Basic)
  U1       C842299    74AHCT125S14-13        Diodes Inc SO-14
  CN1      C108769    XT30UPB-F30.G.Y        XT30 power connector (hand-solder)

Note: replaced original LED part C2890364 (3528 package) with C22464516
(confirmed 5050 package, 5.0x5.0mm, VIH=3.4V confirming level shifter required).

Co-Authored-By: Claude Sonnet 4.6 <noreply@anthropic.com>
Parts:
- C1, C10, C11, C12, C2, C3, C4, C5, C6, C7, C8, C9: LCSC (none) -> C14663; MPN (none) -> CC0603KRX7R9BB104
- C13: LCSC (none) -> C3299; MPN (none) -> GR108M010F12RR0VL4FP0
- D1, D10, D11, D12, D2, D3, D4, D5, D6, D7, D8, D9: LCSC (none) -> C22464516; MPN (none) -> XL-5050RGBWC-WS2812B
- J2: LCSC (none) -> C144394; MPN (none) -> B3B-XH-A(LF)(SN)
- R1: LCSC (none) -> C23138; MPN (none) -> 0603WAF3300T5E
- U1: LCSC (none) -> C842299; MPN (none) -> 74AHCT125S14-13

Commit message: led-indicator: replace CN1 with XT30U-M (male) connector
Switch CN1 from XT30UPB-F (female, C108769) to XT30U-M (male, C99101).
The male connector mates with the battery's female harness plug.

Updated both schematic and PCB:
- Footprint: AMASS_XT30UPB-F → AMASS_XT30U-M (drill 1.8mm → 2.7mm,
  pad size 3×3mm → 3.8×3.8mm, roundrect ratio 0.25 → 0.2)
- LCSC Part: C108769 → C99101
- MPN: XT30UPB-F30.G.Y → XT30U-M
- Refilled copper zones after pad size change; DRC clean (0 errors,
  0 unconnected — only pre-existing C7 library mismatch warning remains)

Co-Authored-By: Claude Sonnet 4.6 <noreply@anthropic.com>
Changed lines of the file:
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@@
 			)
 		)
-		(property "Value" "XT30UPB-F"
+		(property "Value" "XT30U-M"
 			(at 111.76 138.4299 0)
 			(show_name no)
@@
 			)
 		)
-		(property "Footprint" "Connector_AMASS:AMASS_XT30UPB-F_1x02_P5.0mm_Vertical"
+		(property "Footprint" "Connector_AMASS:AMASS_XT30U-M_1x02_P5.0mm_Vertical"
 			(at 116.84 146.05 0)
 			(hide yes)
@@
 			)
 		)
-		(property "Datasheet" "https://lcsc.com/product-detail/Banana-and-Tip-Connectors_Changzhou-Amass-Elec-XT30UPB-F_C108769.html"
+		(property "Datasheet" "https://www.lcsc.com/product-detail/C99101.html"
 			(at 116.84 148.59 0)
 			(hide yes)
@@
 			)
 		)
-		(property "MPN" "XT30UPB-F30.G.Y"
+		(property "MPN" "XT30U-M"
 			(at 116.84 153.67 0)
 			(hide yes)
@@
 			)
 		)
-		(property "LCSC Part" "C108769"
+		(property "LCSC Part" "C99101"
 			(at 116.84 156.21 0)
 			(hide yes)
@@
 			)
 		)
-			(property "LCSC" "C108769"
+			(property "LCSC" "C99101"
 			(at 116.84 137.16 0)
 			(effects (font (size 1.27 1.27)) (hide yes))
 		)
 )
-		(property "LCSC" "C108769"
+		(property "LCSC" "C99101"
 			(at 116.84 137.16 0)
 			(effects
